File: dog tracker rev1.sch (EAGLE design)
At the start: 46 parts, among them IC2 TXB0104, J2 CORTEX_DEBUG_PTH, J6 LiPo, J8 microUSB, Q1 BSS138L, Q2 BSS138L, U2 ATSAMD21G-M, U3 3.3V, X1 LTE-uFL, X2 GNSS-uFL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

Commit message: rev1 fixed and sent to fab
Parts:
- renumbered J2 to SWDPROG
Other:
- note added: "Mike Bales"
- note added: "v1"
- note removed: "Timothy Woo"
- note removed: "v5"
- moved on the sheet: J8
Changed lines of the file:
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@@
 <part name="GND13" library="TimWoo-Aesthetics" library_urn="urn:adsk.eagle:library:502097" deviceset="GND" device=""/>
 <part name="GND14" library="TimWoo-Aesthetics" library_urn="urn:adsk.eagle:library:502097" deviceset="GND" device=""/>
-<part name="J2" library="SparkFun-Connectors" library_urn="urn:adsk.eagle:library:513" deviceset="CORTEX_DEBUG" device="_PTH" package3d_urn="urn:adsk.eagle:package:38290/1"/>
+<part name="SWDPROG" library="SparkFun-Connectors" library_urn="urn:adsk.eagle:library:513" deviceset="CORTEX_DEBUG" device="_PTH" package3d_urn="urn:adsk.eagle:package:38290/1"/>
 </parts>
 <sheets>
 <sheet>
 <plain>
-<text x="419.862" y="6.604" size="3.81" layer="97">v5</text>
-<text x="351.282" y="9.144" size="3.81" layer="97">Timothy Woo</text>
+<text x="419.862" y="6.604" size="3.81" layer="97">v1</text>
+<text x="351.282" y="9.144" size="3.81" layer="97">Mike Bales</text>
 <text x="397.002" y="24.384" size="3.81" layer="97">CC-BY-SA-4.0</text>
 <text x="264.16" y="266.7" size="5.08" layer="94">SIM7000 / micro USB / SIM Card Interface</text>
@@
 </plain>
 <instances>
-<instance part="GND19" gate="1" x="271.78" y="106.68" smashed="yes">
-<attribute name="VALUE" x="269.24" y="104.14" size="1.778" layer="96"/>
-</instance>
-<instance part="J8" gate="G$1" x="261.62" y="116.84" smashed="yes" rot="R180">
-<attribute name="NAME" x="264.16" y="109.22" size="1.778" layer="95" rot="R180"/>
-<attribute name="VALUE" x="264.16" y="127" size="1.778" layer="96" rot="R180"/>
-</instance>
-<instance part="SUPPLY15" gate="G$1" x="271.78" y="127" smashed="yes">
-<attribute name="VALUE" x="270.764" y="130.556" size="1.778" layer="96"/>
+<instance part="GND19" gate="1" x="124.46" y="106.68" smashed="yes">
+<attribute name="VALUE" x="121.92" y="104.14" size="1.778" layer="96"/>
+</instance>
+<instance part="J8" gate="G$1" x="114.3" y="116.84" smashed="yes" rot="R180">
+<attribute name="NAME" x="116.84" y="109.22" size="1.778" layer="95" rot="R180"/>
+<attribute name="VALUE" x="116.84" y="127" size="1.778" layer="96" rot="R180"/>
+</instance>
+<instance part="SUPPLY15" gate="G$1" x="124.46" y="127" smashed="yes">
+<attribute name="VALUE" x="123.444" y="130.556" size="1.778" layer="96"/>
 </instance>
 <instance part="U1" gate="G$1" x="317.5" y="182.88" smashed="yes">
@@
 <attribute name="VALUE" x="30.48" y="160.02" size="1.778" layer="96"/>
 </instance>
-<instance part="J2" gate="G$1" x="71.12" y="116.84" smashed="yes">
+<instance part="SWDPROG" gate="G$1" x="71.12" y="116.84" smashed="yes">
 <attribute name="NAME" x="58.42" y="124.714" size="1.778" layer="95" font="vector"/>
 <attribute name="VALUE" x="58.42" y="106.934" size="1.778" layer="96" font="vector"/>
@@
 <segment>
 <pinref part="GND19" gate="1" pin="GND"/>
-<wire x1="271.78" y1="109.22" x2="271.78" y2="111.76" width="0.1524" layer="91"/>
-<wire x1="271.78" y1="111.76" x2="266.7" y2="111.76" width="0.1524" layer="91"/>
+<wire x1="124.46" y1="109.22" x2="124.46" y2="111.76" width="0.1524" layer="91"/>
+<wire x1="124.46" y1="111.76" x2="119.38" y2="111.76" width="0.1524" layer="91"/>
 <pinref part="J8" gate="G$1" pin="GND"/>
 </segment>
@@
 </segment>
 <segment>
-<pinref part="J2" gate="G$1" pin="GND@3"/>
+<pinref part="SWDPROG" gate="G$1" pin="GND@3"/>
 <wire x1="55.88" y1="119.38" x2="53.34" y2="119.38" width="0.1524" layer="91"/>
 <label x="50.8" y="119.38" size="1.778" layer="95"/>
 </segment>
 <segment>
-<pinref part="J2" gate="G$1" pin="GND@5"/>
+<pinref part="SWDPROG" gate="G$1" pin="GND@5"/>
 <wire x1="55.88" y1="116.84" x2="53.34" y2="116.84" width="0.1524" layer="91"/>
 <label x="50.8" y="116.84" size="1.778" layer="95"/>
@@
 <pinref part="J8" gate="G$1" pin="VBUS"/>
 <pinref part="SUPPLY15" gate="G$1" pin="V_USB"/>
-<wire x1="266.7" y1="121.92" x2="271.78" y2="121.92" width="0.1524" layer="91"/>
-<wire x1="271.78" y1="121.92" x2="271.78" y2="127" width="0.1524" layer="91"/>
+<wire x1="119.38" y1="121.92" x2="124.46" y2="121.92" width="0.1524" layer="91"/>
+<wire x1="124.46" y1="121.92" x2="124.46" y2="127" width="0.1524" layer="91"/>
 </segment>
 <segment>
@@
 <segment>
 <pinref part="J8" gate="G$1" pin="D-"/>
-<wire x1="266.7" y1="119.38" x2="269.24" y2="119.38" width="0.1524" layer="91"/>
-<label x="269.24" y="119.38" size="1.27" layer="95" xref="yes"/>
+<wire x1="119.38" y1="119.38" x2="121.92" y2="119.38" width="0.1524" layer="91"/>
+<label x="121.92" y="119.38" size="1.27" layer="95" xref="yes"/>
 </segment>
 <segment>
@@
 <segment>
 <pinref part="J8" gate="G$1" pin="D+"/>
-<wire x1="266.7" y1="116.84" x2="269.24" y2="116.84" width="0.1524" layer="91"/>
-<label x="269.24" y="116.84" size="1.27" layer="95" xref="yes"/>
+<wire x1="119.38" y1="116.84" x2="121.92" y2="116.84" width="0.1524" layer="91"/>
+<label x="121.92" y="116.84" size="1.27" layer="95" xref="yes"/>
 </segment>
 <segment>
@@
 </segment>
 <segment>
-<pinref part="J2" gate="G$1" pin="!RESET"/>
+<pinref part="SWDPROG" gate="G$1" pin="!RESET"/>
 <wire x1="88.9" y1="111.76" x2="91.44" y2="111.76" width="0.1524" layer="91"/>
 <label x="91.44" y="111.76" size="1.778" layer="95"/>
@@
 </segment>
 <segment>
-<pinref part="J2" gate="G$1" pin="VCC"/>
+<pinref part="SWDPROG" gate="G$1" pin="VCC"/>
 <wire x1="55.88" y1="121.92" x2="53.34" y2="121.92" width="0.1524" layer="91"/>
 <label x="53.34" y="121.92" size="1.778" layer="95"/>
@@
 <net name="N$20" class="0">
 <segment>
-<pinref part="J2" gate="G$1" pin="KEY"/>
+<pinref part="SWDPROG" gate="G$1" pin="KEY"/>
 <wire x1="55.88" y1="114.3" x2="53.34" y2="114.3" width="0.1524" layer="91"/>
 </segment>
@@
 <net name="N$21" class="0">
 <segment>
-<pinref part="J2" gate="G$1" pin="GNDDTCT"/>
+<pinref part="SWDPROG" gate="G$1" pin="GNDDTCT"/>
 <wire x1="55.88" y1="111.76" x2="53.34" y2="111.76" width="0.1524" layer="91"/>
 </segment>
@@
 <net name="N$24" class="0">
 <segment>
-<pinref part="J2" gate="G$1" pin="SWO/TDO"/>
+<pinref part="SWDPROG" gate="G$1" pin="SWO/TDO"/>
 <wire x1="88.9" y1="116.84" x2="91.44" y2="116.84" width="0.1524" layer="91"/>
 </segment>
@@
 <net name="N$25" class="0">
 <segment>
-<pinref part="J2" gate="G$1" pin="NC/TDI"/>
+<pinref part="SWDPROG" gate="G$1" pin="NC/TDI"/>
 <wire x1="88.9" y1="114.3" x2="91.44" y2="114.3" width="0.1524" layer="91"/>
 </segment>
@@
 </segment>
 <segment>
-<pinref part="J2" gate="G$1" pin="SWDCLK/TCK"/>
+<pinref part="SWDPROG" gate="G$1" pin="SWDCLK/TCK"/>
 <wire x1="88.9" y1="119.38" x2="91.44" y2="119.38" width="0.1524" layer="91"/>
 <label x="91.44" y="119.38" size="1.778" layer="95"/>
@@
 </segment>
 <segment>
-<pinref part="J2" gate="G$1" pin="SWDIO/TMS"/>
+<pinref part="SWDPROG" gate="G$1" pin="SWDIO/TMS"/>
 <wire x1="88.9" y1="121.92" x2="91.44" y2="121.92" width="0.1524" layer="91"/>
 <label x="91.44" y="121.92" size="1.778" layer="95"/>

Commit message: rev1 resolved other minor issues, added battery sense, routed all power through LDO and added diode mixing to power input.
Parts:
- removed C5: 0.1uF, TimWoo-Capacitors:CAPMARKED-0603
- added D4, D5: 1A/23V/620mV, SparkFun-DiscreteSemi:DIODE-SCHOTTKY-BAT20J
- added L2: 27nh, rcl:L-USL2012C
- added Q3: BSS138L, TimWoo-MOSFETs:MOSFET-NGENERIC
- added R6: 30k, TimWoo-Resistors:RESISTORMARKED-0603
- added R7, R9: 10k, TimWoo-Resistors:RESISTORMARKED-0603
Connections:
- removed net N$14: C5.2, U2.GNDANA
- removed net N$21: SWDPROG.GNDDTCT
- new net BATT_SENSE: R6.2, R7.1, U2.PB03(AIN11/SER5:1)
- new net N$15: Q3.D, R6.1
- new net N$19: D4.C, D5.C, R4.1, U3.IN
- new net SENSE_GATE: Q3.G, U2.PA12(I2C/SER2:0+)
- new net V_BATT: D5.A, J6.1, R7.2
- net 3.3V: now also L2.1, R9.2; no longer J6.1
- net GND: now also Q3.S, SWDPROG.GNDDTCT, U2.GNDANA; no longer C5.1
- net SWDIO: now also R9.1
- net VDDANA: now also L2.2
- net V_USB: now also D4.A; no longer R4.1, U3.IN
Other:
- moved on the sheet: H1, H2, R4
